File: Hardware/night-light.brd (EAGLE design)
At the start: 17.8 x 33 mm, 52 parts, among them Q1 8/16/20MHz, U1 ATMEGA328, U2 MIC5205

Commit message: added tlc5947
Parts:
- added IREF_R4: 3.3K, eagle-ltspice:R0603
- added TP_SOUT: TPTP20R, testpad:TP20R
Connections:
- removed net CLK: U1.9
- removed net D3: U1.1
- removed net D7: U1.11
- removed net LAT: U1.10
- new net BLANK: U$2.30, U1.11
- new net N$30: LED3.C, U$2.23
- new net N$31: LED2.C, U$2.24
- new net SCLK: U$2.31, U1.1
- new net XLAT: U$2.26, U1.10
- net 3.3V: now also LED10.A, LED11.A, LED12.A, LED13.A, LED14.A, LED15.A, LED16.A, LED17.A, LED18.A, LED19.A, LED2.A, LED20.A, LED21.A, LED22.A, LED23.A, LED24.A, LED25.A, LED3.A, LED4.A, LED5.A, LED6.A, LED7.A, LED8.A, LED9.A
- net GND: now also IREF_R4.2
- net N$10: now also LED23.C, U$2.3; no longer LED6.A, U$2.5
- net N$11: now also LED22.C, U$2.4; no longer LED7.A, U$2.6
- net N$12: now also LED21.C, U$2.5; no longer LED8.A, U$2.7
- net N$13: now also LED20.C, U$2.6; no longer LED9.A, U$2.8
- net N$14: now also LED19.C, U$2.7; no longer LED10.A, U$2.9
- net N$15: now also LED18.C, U$2.8; no longer LED11.A, U$2.10
- net N$16: now also LED17.C, U$2.9; no longer LED12.A, U$2.11
- net N$17: now also LED16.C, U$2.10; no longer LED13.A, U$2.12
- net N$18: now also LED15.C, U$2.11; no longer LED14.A, U$2.13
- net N$19: now also LED14.C, U$2.12; no longer LED15.A, U$2.14
- net N$20: now also LED13.C, U$2.13; no longer LED16.A, U$2.15
- net N$21: now also LED12.C, U$2.14; no longer LED17.A, U$2.16
- net N$22: now also LED11.C, U$2.15; no longer LED18.A, U$2.17
- net N$23: now also LED10.C, U$2.16; no longer LED19.A, U$2.18
- net N$24: now also LED9.C, U$2.17; no longer LED20.A, U$2.19
- net N$25: now also LED8.C, U$2.18; no longer LED21.A, U$2.20
- net N$26: now also LED7.C, U$2.19; no longer LED22.A, U$2.21
- net N$27: now also LED6.C, U$2.20; no longer LED23.A, U$2.22
- net N$28: now also LED5.C, U$2.21; no longer LED24.A, U$2.23
- net N$29: now also LED4.C, U$2.22; no longer LED25.A, U$2.24
- net N$5: now also LED25.C; no longer LED2.A
- net N$6: now also IREF_R4.1, U$2.27; no longer LED3.A, U$2.2
- net N$8: now also LED24.C, U$2.2; no longer LED4.A, U$2.3
- net N$9: now also TP_SOUT.TP, U$2.25; no longer LED5.A, U$2.4
Routing:
- net SCLK: track 0.00 -> 11.3 mm, vias 0 -> 1
- net D3: track 11.3 -> 0.00 mm, vias 1 -> 0
- net D7: track 6.99 -> 0.00 mm
- net BLANK: track 0.00 -> 6.99 mm
- net XLAT: track 0.00 -> 4.79 mm
- net LAT: track 4.79 -> 0.00 mm
- net CLK: track 2.84 -> 0.00 mm

Commit message: new pcb
Parts:
- removed C19: 10uF, SparkFun:EIA3216
- removed C3: 0.1uF, SparkFun:0603-CAP
- removed FRAME1: FRAME-LETTER, SparkFun-Aesthetics:CREATIVE_COMMONS
- removed JP2, JP3: (no value), SparkFun:1X02
- removed LED1: Red, Testing:0603-LED-ALT1
- removed R1, R3: (no value), SparkFun:0603-RES
- removed R11: 10K, SparkFun:0603-RES
- removed SJ1: (no value), SparkFun-Passives:SJ_2S
- removed U$1: LOGO-SFESK, SparkFun:SFE-LOGO-FLAME
- removed U$11: LOGO-SFENEW, SparkFun:SFE-NEW-WEBLOGO
- removed U$3: OSHW-LOGOS, SparkFun:OSHW-LOGO-S
- removed U2: MIC5205, SparkFun:SOT23-5
- added C6, C7: 4.7uF, SparkFun-Capacitors:0603-CAP
- added D1: RED, SparkFun-LED:LED-0603
- added JP4: M02PTH, SparkFun-Connectors:1X02
- added JP6: Micro USB, SparkFun-Connectors:USB-AB-MICRO-SMD_V03
- added JP7: JST, SparkFun-Connectors:JST-2-SMD
- added R5: 330, SparkFun-Resistors:0603-RES
- added R7: 2.0k, SparkFun-Resistors:0603-RES
- added R8: (no value), SparkFun-Resistors:AXIAL-0.1EZ
- added U4: MCP73831, SparkFun-PowerIC:SOT23-5
- moved LED13 111.6 mm to (-47.0, 22.9)
- moved LED12 106.8 mm to (-39.4, 22.9)
- moved LED23 105.9 mm to (-48.3, 34.3)
- moved LED18 104.8 mm to (-48.3, 29.2)
- moved LED17 97.9 mm to (-40.6, 29.2)
- moved LED22 97.5 mm to (-40.6, 34.3)
- moved LED4 94.0 mm to (-52.1, 39.4)
- moved LED16 91.5 mm to (-33.0, 29.2)
- moved LED21 89.3 mm to (-33.0, 34.3)
- moved LED9 88.4 mm to (-41.9, 44.5)
- moved LED25 88.2 mm to (-25.4, 39.4)
- moved LED3 88.0 mm to (-45.7, 39.4)
- moved LED15 85.5 mm to (-25.4, 29.2)
- moved LED2 82.3 mm to (-39.4, 39.4)
- moved LED11 81.9 mm to (-33.0, 39.4)
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Connections:
- net AREF renamed N$32
- removed net A4: JP2.1, R1.1, U1.27
- removed net A5: JP2.2, R3.1, U1.28
- removed net N$3: LED1.A, SJ1.1, U2.5
- removed net N$4: LED1.C, R11.2
- removed net RAW: C19.A, U2.1, U2.3
- new net 5V: C6.1, JP6.VBUS1, R5.2, U4.4
- new net N$34: D1.A, R5.1
- new net PROG1: R7.1, R8.P$2, U4.5
- new net STAT1: D1.C, U4.1
- net A6: no longer JP3.1
- net A7: no longer JP3.2
- net GND: now also C6.2, C7.2, JP4.1, JP6.GND1, JP7.1, R7.2, R8.P$1, U4.2; no longer C19.C, C3.1, R11.1, U2.2
- net VCC: now also C7.1, JP4.2, JP7.2, U4.3; no longer C3.2, R1.2, R3.2, SJ1.2
Routing:
- net RESET: track 57.0 -> 0.00 mm, vias 2 -> 0
- net VCC: track 56.8 -> 0.00 mm, vias 2 -> 0
- net RXI: track 40.2 -> 0.00 mm, vias 1 -> 0
- net D10: track 24.4 -> 0.00 mm, vias 1 -> 0
- net TXO: track 24.1 -> 0.00 mm
- net N$32: track 22.8 -> 0.00 mm, vias 2 -> 0
- net MISO: track 19.5 -> 0.00 mm, vias 1 -> 0
- net A5: track 14.1 -> 0.00 mm, vias 1 -> 0
- net D9: track 11.7 -> 0.00 mm
- net MOSI: track 11.7 -> 0.00 mm, vias 1 -> 0
- net RAW: track 11.3 -> 0.00 mm, vias 2 -> 0
- net SCLK: track 11.3 -> 0.00 mm, vias 1 -> 0
- net DIN: track 10.1 -> 0.00 mm, vias 1 -> 0
- net SCK: track 9.42 -> 0.00 mm
- net GND: track 9.36 -> 0.00 mm, vias 13 -> 0
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- removed copper zone on layer 1, net GND
- removed copper zone on layer 16, net GND
Other:
- board size 17.8 x 33 mm -> 50 x 50 mm
- board text removed: "10"
- board text removed: "10MHz"
- board text removed: "11"
- board text removed: "12"
- board text removed: "13"
- board text removed: "168 / 5V Reg / 16MHz"
- board text removed: "168 / 5V Reg / 20MHz"
- board text removed: "168V / 3.3V Reg / 8MHz"
- board text removed: "16MHz"
- board text removed: "2"
- board text removed: "20MHz"
- board text removed: "3"
- board text removed: "3.3V"
- board text removed: "4"
- board text removed: "5"
- board text removed: "5V"
- board text removed: "6"
- board text removed: "7"
- board text removed: "8"
- board text removed: "8MHz"
- board text removed: "9"
- board text removed: "A0"
- board text removed: "A1"
- board text removed: "A2"
- board text removed: "A3"
- board text removed: "A4"
- board text removed: "A5"
- board text removed: "A6"
- board text removed: "A7"
- board text removed: "Arduino Pro"
- board text removed: "Arduino Pro Mini"
- board text removed: "BLK"
- board text removed: "GND"
- board text removed: "GRN"
- board text removed: "Mark back accordingly"
- board text removed: "Mini"
- board text removed: "Original Arduino Mini Design by Team Arduino Arduino Pro Mini Design by SparkFun Electronics Revised by Pete Lewis"
- board text removed: "RAW"
- board text removed: "RST"
- board text removed: "RXI"
- board text removed: "Reset"
- board text removed: "TXO"
- board text removed: "VCC"
- board text removed: "Valid combinations:"
- board text removed: "v14"
- board text removed: "www.arduino.cc"
